File: ergogen/pcbs/clyde.kicad_pcb (KiCad board)
At the start: 2 copper layers, 114.3 x 83.3 mm, 60 parts

Commit message: finish routing
Connections:
- U0 pad 5: matrix_ring_top -> matrix_ring_bottom
- U0 pad 7: matrix_ring_bottom -> matrix_ring_top
Changed lines of the file:
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@@
     (pad "3" thru_hole rect (at 8.82 -19.05) (size 1.84 1.7) (drill oval 1.16 1.02) (layers *.Cu *.Mask) (net 2 "GND"))
     (pad "4" thru_hole oval (at 8.82 -16.51) (size 1.84 1.7) (drill oval 1.16 1.02) (layers *.Cu *.Mask) (net 1 "matrix_pinky_bottom"))
-    (pad "5" thru_hole oval (at 8.82 -13.97) (size 1.84 1.7) (drill oval 1.16 1.02) (layers *.Cu *.Mask) (net 7 "matrix_ring_top"))
+    (pad "5" thru_hole oval (at 8.82 -13.97) (size 1.84 1.7) (drill oval 1.16 1.02) (layers *.Cu *.Mask) (net 5 "matrix_ring_bottom"))
     (pad "6" thru_hole oval (at 8.82 -11.43) (size 1.84 1.7) (drill oval 1.16 1.02) (layers *.Cu *.Mask) (net 6 "matrix_ring_home"))
-    (pad "7" thru_hole oval (at 8.82 -8.89) (size 1.84 1.7) (drill oval 1.16 1.02) (layers *.Cu *.Mask) (net 5 "matrix_ring_bottom"))
+    (pad "7" thru_hole oval (at 8.82 -8.89) (size 1.84 1.7) (drill oval 1.16 1.02) (layers *.Cu *.Mask) (net 7 "matrix_ring_top"))
     (pad "8" thru_hole rect (at 8.82 -6.35) (size 1.84 1.7) (drill oval 1.16 1.02) (layers *.Cu *.Mask) (net 2 "GND"))
     (pad "9" thru_hole oval (at 8.82 -3.81) (size 1.84 1.7) (drill oval 1.16 1.02) (layers *.Cu *.Mask) (net 10 "matrix_middle_top"))
