File: prod/clyde-switch-plate.kicad_pcb (KiCad board)
At the start: 2 copper layers, 114.3 x 83.3 mm, 0 parts

Commit message: set to JLC
Other:
- outline, holes or cut-outs redrawn
Changed lines of the file:
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@@
   (page A3)
   (title_block
-    (title clyde-plate)
+    (title clyde-switch-plate)
     (rev 1.0.0)
     (company sboysel)
@@
     (add_net "")
   )
-            (gr_line (start 142.875 159.925) (end 142.875 106.77499999999999) (angle 90) (layer Edge.Cuts) (width 0.15))
+            (gr_line (start 142.875 161.425) (end 142.875 106.77499999999999) (angle 90) (layer Edge.Cuts) (width 0.15))
 (gr_line (start 144.875 104.77499999999999) (end 236.12500000000003 104.77499999999999) (angle 90) (layer Edge.Cuts) (width 0.15))
 (gr_line (start 238.12500000000003 106.77499999999999) (end 238.12500000000003 159.925) (angle 90) (layer Edge.Cuts) (width 0.15))
@@
 (gr_line (start 257.175 163.925) (end 257.175 186.11875) (angle 90) (layer Edge.Cuts) (width 0.15))
 (gr_line (start 255.175 188.11875) (end 199.64375 188.11875) (angle 90) (layer Edge.Cuts) (width 0.15))
-(gr_line (start 197.64375 186.11875) (end 197.64375 163.925) (angle 90) (layer Edge.Cuts) (width 0.15))
-(gr_line (start 195.64375 161.925) (end 144.875 161.925) (angle 90) (layer Edge.Cuts) (width 0.15))
+(gr_line (start 197.64375 186.11875) (end 197.64375 165.425) (angle 90) (layer Edge.Cuts) (width 0.15))
+(gr_line (start 195.64375 163.425) (end 144.875 163.425) (angle 90) (layer Edge.Cuts) (width 0.15))
 (gr_arc (start 144.875 106.77499999999999) (end 144.875 104.77499999999999) (angle -90) (layer Edge.Cuts) (width 0.15))
 (gr_arc (start 236.12500000000003 106.77499999999999) (end 238.12500000000003 106.77499999999999) (angle -90) (layer Edge.Cuts) (width 0.15))
@@
 (gr_arc (start 255.175 186.11875) (end 255.175 188.11875) (angle -90) (layer Edge.Cuts) (width 0.15))
 (gr_arc (start 199.64375 186.11875) (end 197.64375 186.11875) (angle -90) (layer Edge.Cuts) (width 0.15))
-(gr_arc (start 195.64375 163.925) (end 197.64375 163.925) (angle -90) (layer Edge.Cuts) (width 0.15))
-(gr_arc (start 144.875 159.925) (end 142.875 159.925) (angle -90) (layer Edge.Cuts) (width 0.15))
+(gr_arc (start 195.64375 165.425) (end 197.64375 165.425) (angle -90) (layer Edge.Cuts) (width 0.15))
+(gr_arc (start 144.875 161.425) (end 142.875 161.425) (angle -90) (layer Edge.Cuts) (width 0.15))
 (gr_line (start 145.4 159.4) (end 159.4 159.4) (angle 90) (layer Edge.Cuts) (width 0.15))
 (gr_line (start 159.4 159.4) (end 159.4 145.4) (angle 90) (layer Edge.Cuts) (width 0.15))
